File: design/hackpad.kicad_sch (KiCad schematic)
At the start: 38 parts, among them SW1 SW_Push, SW10 RotaryEncoder, SW2 SW_Push, SW3 SW_Push, SW4 SW_Push, SW5 SW_Push, SW6 SW_Push, SW7 SW_Push, SW8 SW_Push, SW9 SW_Push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

Commit message: add firmware, forgor to add the 5v net
Parts:
- added H1, H2, H3, H4: MountingHole, MountingHole:MountingHole_2.1mm, symbol Mechanical:MountingHole
- D10, D11, D12, D13, D14, D15, D16, D17, D18: footprint LED_SMD:LED_SK6812MINI-E_3.2x2.8mm_P1.5mm_ReverseMount -> LED_SMD:LED_SK6812MINI_PLCC4_3.5x3.5mm_P1.75mm
Connections:
- net +3V3: now also U1.26 (3V3_1)
- net 5V: now reaches U1.14 (VBUS)
